Commit message: rviz file to test driving of robot

File: description/robot.urdf.xacro (robot description, xacro)
@@ -2,3 +2,4 @@
 <robot xmlns:xacro="http://www.ros.org/wiki/xacro"  name="robot">
     <xacro:include filename="robot_core.xacro"/>
+    <xacro:include filename="gazebo_control.xacro"/>
 </robot>

File: description/robot_core.xacro (robot description, xacro)
@@ -27,7 +27,10 @@
     </collision>
     <xacro:inertial_box mass="0.5" x="0.3" y="0.3" z="0.15">
-      <origin xyz="0.15 0 0.075"/>
+      <origin xyz="0.15 0 0.075" rpy="0 0 0"/>
     </xacro:inertial_box>
   </link>
+  <gazebo reference="chassis">
+    <material>Gazebo/White</material>
+  </gazebo>
   <!-- LEFT WHEEL LINK-->
   <joint name="left_wheel_joint" type="continuous">
@@ -53,9 +56,12 @@
     </xacro:inertial_cylinder>
   </link>
+  <gazebo reference="left_wheel">
+    <material>Gazebo/Blue</material>
+  </gazebo>
   <!-- RIGHT WHEEL LINK-->
   <joint name="right_wheel_joint" type="continuous">
     <parent link="base_link"/>
     <child link="right_wheel"/>
-    <origin xyz="0 -0.175 0" rpy="-${pi/2} 0 0"/>
+    <origin xyz="0 -0.175 0" rpy="${pi/2} 0 0"/>
     <axis xyz="0 0 -1"/>
   </joint>
@@ -76,4 +82,7 @@
     </xacro:inertial_cylinder>
   </link>
+  <gazebo reference="right_wheel">
+    <material>Gazebo/Blue</material>
+  </gazebo>
   <!-- CASTER WHEEL LINK-->
   <joint name="caster_wheel_joint" type="fixed">
@@ -98,3 +107,8 @@
     </xacro:inertial_sphere>
   </link>
+  <gazebo reference="caster_wheel">
+    <material>Gazebo/Black</material>
+    <mu1 value="0.001"/>
+    <mu2 value="0.001"/>
+  </gazebo>
 </robot>
