Commit message: Updated files

File: description/materials.xacro (robot description, xacro)
@@ -13,3 +13,6 @@
     <color rgba="0 0 0 1"/>
   </material>
+  <material name="red">
+    <color rgba="1 0 0 1"/>
+  </material>
 </robot>

File: description/robot.urdf.xacro (robot description, xacro)
@@ -3,3 +3,5 @@
     <xacro:include filename="robot_core.xacro"/>
     <xacro:include filename="gazebo_control.xacro"/>
+    <xacro:include filename="lidar.xacro"/>
+    <xacro:include filename="camera.xacro"/>
 </robot>

File: description/robot_core.xacro (robot description, xacro)
@@ -112,3 +112,29 @@
     <mu2 value="0.001"/>
   </gazebo>
+  <!-- LIDAR -->
+  <joint name="lidar_joint" type="fixed">
+      <parent link="chassis"/>
+      <child link="lidar_link"/>
+      <origin xyz="0.1 0 0.175" rpy="0 0 0"/>
+      <axis xyz="0 1 0" rpy="0 0 0"/>
+  </joint>
+  <link name="lidar_link">
+    <visual>
+      <geometry>
+        <cylinder radius="0.05" length="0.04"/>
+      </geometry>
+      <material name="red"/>
+    </visual>
+    <collision>
+      <geometry>
+          <cylinder radius="0.05" length="0.04"/>
+      </geometry>
+    </collision>
+    <xacro:inertial_cylinder mass="0.1" length="0.04" radius="0.05">
+      <origin xyz="0 0 0" rpy="0 0 0"/>
+    </xacro:inertial_cylinder>
+  </link>
+  <gazebo reference="lidar_link">
+    <material>Gazebo/Red</material>
+  </gazebo>
 </robot>
